Commit message: primera edicion del urdf

File: objects/hermesArm.urdf (robot description, URDF)
Before this commit: robot hermesArm, 1 links, 0 joints
Links:
- removed link Base
- added link base
- added link link1
- added link link2
- added link link3
- added link link4
- added link link5
- added link link6
- added link link7
Joints:
- added joint joint1: type revolute, parent base, child link1, origin xyz=-2 5 0 rpy=0 0 1.57, limit lower=-3.14 upper=3.14 effort=100 velocity=100
- added joint joint2: type revolute, parent link1, child link2, limit lower=-1.83 upper=1.83 effort=100 velocity=100
- added joint joint3: type revolute, parent link2, child link3, limit lower=-3.14 upper=3.14 effort=100 velocity=100
- added joint joint4: type revolute, parent link3, child link4, limit lower=-1.83 upper=1.83 effort=100 velocity=100
- added joint joint5: type revolute, parent link4, child link5, limit lower=-3.14 upper=3.14 effort=100 velocity=100
- added joint joint6: type revolute, parent link5, child link6, limit lower=-1.83 upper=1.83 effort=100 velocity=100
- added joint joint7: type revolute, parent link6, child link7, limit lower=-3.14 upper=3.14 effort=100 velocity=100

Commit message: Terminado el primer modelo urdf

File: objects/hermesArm.urdf (robot description, URDF)
Before this commit: robot hermesArm, 8 links, 7 joints
Joints:
- joint joint1: axis (none) -> 0 0 1; origin xyz=-2 5 0 rpy=0 0 1.57 -> xyz=0 0 -0.3060 rpy=1.5708 0 0
- joint joint2: axis (none) -> 0 0 1; origin (none) -> xyz=0 0 0 rpy=-1.5708 0 0
- joint joint3: axis (none) -> 0 0 1; origin (none) -> xyz=0 0 -0.391 rpy=1.5708 0 0
- joint joint4: origin (none) -> xyz=0 0 0 rpy=-1.5708 0 0
- joint joint5: axis (none) -> 0 0 1; origin (none) -> xyz=0 0 -0.2975 rpy=1.5708 0 0
- joint joint6: origin (none) -> xyz=0 0 0 rpy=-1.5708 0 0
- joint joint7: axis (none) -> 0 0 1; origin (none) -> xyz=0 0 -0.3045 rpy=3.1416 0 0
