Commit message: working on scenario

File: urdf/hermesArm.urdf (robot description, URDF)
Before this commit: robot hermesArm, 8 links, 7 joints
Joints:
- joint joint1: axis 0 0 1 -> 0 1 0; origin xyz=0 0 -0.3060 rpy=1.5708 0 0 -> xyz=0 0 -0.3060 rpy=1.5707963267949 0 0
- joint joint2: axis 0 0 1 -> 0 -1 0; origin xyz=0 0 0 rpy=-1.5708 0 0 -> xyz=0 0 0 rpy=-1.5707963267949 0 0
- joint joint3: axis 0 0 1 -> 0 1 0; origin xyz=0 0 -0.391 rpy=1.5708 0 0 -> xyz=0 0 -0.391 rpy=1.5707963267949 0 0
- joint joint4: axis (none) -> 0 -1 0; origin xyz=0 0 0 rpy=-1.5708 0 0 -> xyz=0 0 0 rpy=-1.5707963267949 0 0
- joint joint5: axis 0 0 1 -> 0 1 0; origin xyz=0 0 -0.2975 rpy=1.5708 0 0 -> xyz=0 0 -0.2975 rpy=1.5707963267949 0 0
- joint joint6: axis (none) -> 0 -1 0; origin xyz=0 0 0 rpy=-1.5708 0 0 -> xyz=0 0 0 rpy=-1.5707963267949 0 0
- joint joint7: axis 0 0 1 -> 0 0 -1
